File: ortho_40%_split/left_hand/ortho_40_left.kicad_pcb (KiCad board)
At the start: 2 copper layers, 112 x 79 mm, 90 parts, among them J1 prog_pins, J2 Conn_01x01, J3 Conn_01x01, J5 Conn_01x01, J7 Conn_01x01, J8 Conn-Battery, U1 cargador-USB, U2 HOLE, U2 core51822, U3 HOLE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

Commit message: working on right hand
Parts:
- removed the U2 at (39.4, 85.5)
- removed the U3 at (115.7, 85.6)
- J2, J3, J5, J7: footprint Mounting_Holes:MountingHole_3.2mm_M3_ISO14580_Pad -> keyboard_parts:HOLE_M3
- K-11, K-12, K-13, K-14, K-15, K-16, K-21, K-22, K-23, K-24, K-25, K-26, K-31, K-32, K-33, K-34, K-35, K-36, K-41, K-42, K-43, K-44, K-45, K-46: footprint MX_Alps_Hybrid:MX-1U-NoLED -> Keebio:Hybrid_PCB_100H_Dual_hole
- moved ? 38.2 mm to (59.4, 64.2), turned to 20 degrees
- moved SW-RESET1 1.15 mm to (47.4, 63.6)
- moved R1 0.84 mm to (96.2, 35.4)
- moved D14 0.83 mm to (93.7, 35.4)
- moved J5 0.47 mm to (37.7, 84.9)
Routing:
- net GND: track 24.9 -> 48.8 mm, vias 7 -> 12
- net VCC: track 376.5 -> 356.9 mm, vias 18 -> 13
- net Net-(LED1-Pad4): track 50.2 -> 55.6 mm
- net col-1: track 133.6 -> 137.9 mm
- net col-2: track 109.7 -> 105.9 mm
- net row-1: track 101.2 -> 97.5 mm
- net Net-(D14-Pad2): track 10.2 -> 6.72 mm
- net Net-(D26-Pad2): track 12.8 -> 15.7 mm
- net (no net): track 2.81 -> 0.00 mm
- net LED-G: track 33.2 -> 35.4 mm
- net Net-(D11-Pad2): track 5.87 -> 7.68 mm
- net Net-(LED1-Pad2): track 19.5 -> 18.2 mm
- net Net-(LED2-Pad2): track 19.2 -> 17.9 mm
- net underglow: track 8.87 -> 7.84 mm
- net Net-(D34-Pad2): track 12.1 -> 13.0 mm
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Other:
- board text added: "ortho_40_left v0.3 22/07/2018 by Bananacocodrilo"
- board text removed: "ortho_40_left v0.2 18/07/2018 by Bananacocodrilo"
